File: Electrical/microtaur-teensy41.sch (KiCad schematic (older format))
At the start: 33 parts, among them J1 Conn_01x06, J2 USB_A, U1 Teensy4.1, U3 LM7805_TO220

Commit message: Add files via upload
Parts:
- removed J1: Conn_01x06, Connector_JST:JST_SH_SM06B-SRSS-TB_1x06-1MP_P1.00mm_Horizontal, symbol Connector_Generic:Conn_01x06
- C1: Part Number (none) -> 2679-C0805X7R500-22MNETR-ND; URL (none) -> https://www.digikey.com/en/products/detail/venkel/C0805X7R5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
- IMU1: Part Number (none) -> 455-1790-2-ND; URL (none) -> https://www.digikey.com/en/products/detail/jst-sales-americ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
- J2: Part Number (none) -> WM8672-ND; URL (none) -> https://www.digikey.com/en/products/detail/molex/1050570001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
- MPOW1, MPOW2, MPOW3, MPOW4, MPOW5, MPOW6, MPOW7, MPOW8, PWR1: URL (none) -> https://hobbyking.com/en_us/xt30u-m-f-male-female-5pairs-pe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
- R1: Part Number (none) -> 541-2795-2-ND; URL (none) -> https://www.digikey.com/en/products/detail/vishay-dale/RCS0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
- R2: Part Number (none) -> 541-RCS06032K49FKEATR-ND; URL (none) -> https://www.digikey.com/en/products/detail/vishay-dale/RCS0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
- SER1, SER2, SER3, SER4, SER5, SER6, SER7, SER8: Part Number (none) -> 455-1803-2-ND; URL (none) -> https://www.digikey.com/en/products/detail/jst-sales-americ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
- U1: URL (none) -> https://www.pjrc.com/store/teensy41.html
- U3: footprint Package_TO_SOT_THT:TO-220-3_Horizontal_TabDown -> Package_TO_SOT_SMD:SOT-223; Part Number (none) -> NCP1117LPST33T3COSTR-ND; URL (none) -> https://www.digikey.com/en/products/detail/on-semiconductor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
