File: Electrical/microtaur-teensy41.sch (KiCad schematic (older format))
At the start: 33 parts, among them J1 Conn_01x06, J2 USB_A, U1 Teensy4.1, U3 LM7805_TO220

Commit message: updated solidworks model
Parts:
- C1: symbol Device:C_Small -> microtaur-teensy41-rescue:C_Small-Device
- H1, H2, H3, H4, H5, H6, H7, H8: symbol Mechanical:MountingHole -> microtaur-teensy41-rescue:MountingHole-Mechanical
- IMU1: symbol Connector_Generic:Conn_01x04 -> microtaur-teensy41-rescue:Conn_01x04-Connector_Generic
- J1: symbol Connector_Generic:Conn_01x06 -> microtaur-teensy41-rescue:Conn_01x06-Connector_Generic
- MPOW1, MPOW2, MPOW3, MPOW4, MPOW5, MPOW6, MPOW7, MPOW8, PWR1: symbol Connector_Generic:Conn_01x02 -> microtaur-teensy41-rescue:Conn_01x02-Connector_Generic
- R1, R2: symbol Device:R_Small -> microtaur-teensy41-rescue:R_Small-Device
- SER1, SER2, SER3, SER4, SER5, SER6, SER7, SER8: symbol Connector_Generic:Conn_01x03 -> microtaur-teensy41-rescue:Conn_01x03-Connector_Generic
- U3: symbol Regulator_Linear:LM7805_TO220 -> microtaur-teensy41-rescue:LM7805_TO220-Regulator_Linear
Changed lines of the file:
@@
 SDA
 $Comp
-L Device:R_Small R1
+L microtaur-teensy41-rescue:R_Small-Device R1
 U 1 1 6093F1E2
 P 10100 5550
@@
 $EndComp
 $Comp
-L Device:R_Small R2
+L microtaur-teensy41-rescue:R_Small-Device R2
 U 1 1 6093F5F8
 P 10100 5750
@@
 $EndComp
 $Comp
-L power:GND #PWR0110
+L microtaur-teensy41-rescue:GND-power #PWR0110
 U 1 1 6093F92D
 P 10100 5850
@@
 BAT_MON
 $Comp
-L Connector_Generic:Conn_01x06 J1
+L microtaur-teensy41-rescue:Conn_01x06-Connector_Generic J1
 U 1 1 6094B3D5
 P 7850 5450
@@
 PS2_CLK
 $Comp
-L power:GND #PWR0111
+L microtaur-teensy41-rescue:GND-power #PWR0111
 U 1 1 60968EE0
 P 5750 6050
@@
 Connection ~ 9500 5450
 $Comp
-L Device:C_Small C1
+L microtaur-teensy41-rescue:C_Small-Device C1
 U 1 1 60984EAC
 P 9500 5550
@@
 GND
 $Comp
-L power:GND #PWR0108
+L microtaur-teensy41-rescue:GND-power #PWR0108
 U 1 1 6091D001
 P 10300 4250
@@
 	9950 4050 10300 4050
 $Comp
-L power:GND #PWR0107
+L microtaur-teensy41-rescue:GND-power #PWR0107
 U 1 1 6091C656
 P 10300 3850
@@
 	9950 3650 10300 3650
 $Comp
-L power:GND #PWR0106
+L microtaur-teensy41-rescue:GND-power #PWR0106
 U 1 1 6091BA78
 P 10300 3450
@@
 	9950 3250 10300 3250
 $Comp
-L power:GND #PWR0105
+L microtaur-teensy41-rescue:GND-power #PWR0105
 U 1 1 6091B106
 P 10300 3050
@@
 	9950 2850 10300 2850
 $Comp
-L power:GND #PWR0104
+L microtaur-teensy41-rescue:GND-power #PWR0104
 U 1 1 6091A8BE
 P 10300 2650
@@
 	9950 2450 10300 2450
 $Comp
-L power:GND #PWR0103
+L microtaur-teensy41-rescue:GND-power #PWR0103
 U 1 1 60919F5E
 P 10300 2250
@@
 	9950 2050 10300 2050
 $Comp
-L power:GND #PWR0102
+L microtaur-teensy41-rescue:GND-power #PWR0102
 U 1 1 609186A5
 P 10300 1850
@@
 $EndComp
 $Comp
-L power:GND #PWR0101
+L microtaur-teensy41-rescue:GND-power #PWR0101
 U 1 1 6091811A
 P 10300 1450
@@
 	9950 1250 10300 1250
 $Comp
-L Connector_Generic:Conn_01x03 SER7
+L microtaur-teensy41-rescue:Conn_01x03-Connector_Generic SER7
 U 1 1 60916A47
 P 10500 3750
@@
 $EndComp
 $Comp
-L Connector_Generic:Conn_01x03 SER1
+L microtaur-teensy41-rescue:Conn_01x03-Connector_Generic SER1
 U 1 1 6090E039
 P 10500 1350
@@
 $EndComp
 $Comp
-L Connector_Generic:Conn_01x03 SER2
+L microtaur-teensy41-rescue:Conn_01x03-Connector_Generic SER2
 U 1 1 6090D835
 P 10500 1750
@@
 $EndComp
 $Comp
-L Connector_Generic:Conn_01x03 SER6
+L microtaur-teensy41-rescue:Conn_01x03-Connector_Generic SER6
 U 1 1 6090CC6A
 P 10500 3350
@@
 $EndComp
 $Comp
-L Connector_Generic:Conn_01x03 SER3
+L microtaur-teensy41-rescue:Conn_01x03-Connector_Generic SER3
 U 1 1 6090CC64
 P 10500 2150
@@
 $EndComp
 $Comp
-L Connector_Generic:Conn_01x03 SER8
+L microtaur-teensy41-rescue:Conn_01x03-Connector_Generic SER8
 U 1 1 608A52BA
 P 10500 4150
@@
 $EndComp
 $Comp
-L Connector_Generic:Conn_01x03 SER5
+L microtaur-teensy41-rescue:Conn_01x03-Connector_Generic SER5
 U 1 1 608A4971
 P 10500 2950
@@
 $EndComp
 $Comp
-L Connector_Generic:Conn_01x03 SER4
+L microtaur-teensy41-rescue:Conn_01x03-Connector_Generic SER4
 U 1 1 608A46A8
 P 10500 2550
@@
 $EndComp
 $Comp
-L power:GND #PWR0109
+L microtaur-teensy41-rescue:GND-power #PWR0109
 U 1 1 6093DB86
 P 10800 5750
@@
 $EndComp
 $Comp
-L Connector_Generic:Conn_01x02 PWR1
+L microtaur-teensy41-rescue:Conn_01x02-Connector_Generic PWR1
 U 1 1 608ADE78
 P 11000 5750
@@
 $EndComp
 $Comp
-L power:Vdrive #PWR0112
+L microtaur-teensy41-rescue:Vdrive-power #PWR0112
 U 1 1 608AFDF3
 P 9500 5450
@@
 $EndComp
 $Comp
-L Mechanical:MountingHole H3
+L microtaur-teensy41-rescue:MountingHole-Mechanical H3
 U 1 1 608B7434
 P 750 7250
@@
 $EndComp
 $Comp
-L Mechanical:MountingHole H7
+L microtaur-teensy41-rescue:MountingHole-Mechanical H7
 U 1 1 608B8276
 P 1000 7250
@@
 $EndComp
 $Comp
-L Mechanical:MountingHole H8
+L microtaur-teensy41-rescue:MountingHole-Mechanical H8
 U 1 1 608B8652
 P 1000 7450
@@
 $EndComp
 $Comp
-L Mechanical:MountingHole H4
+L microtaur-teensy41-rescue:MountingHole-Mechanical H4
 U 1 1 608B8ABD
 P 750 7450
@@
 $EndComp
 $Comp
-L Mechanical:MountingHole H2
+L microtaur-teensy41-rescue:MountingHole-Mechanical H2
 U 1 1 608B8C2F
 P 750 7000
@@
 $EndComp
 $Comp
-L Mechanical:MountingHole H6
+L microtaur-teensy41-rescue:MountingHole-Mechanical H6
 U 1 1 608B8EC9
 P 1000 7000
@@
 $EndComp
 $Comp
-L Mechanical:MountingHole H5
+L microtaur-teensy41-rescue:MountingHole-Mechanical H5
 U 1 1 608B9277
 P 1000 6800
@@
 $EndComp
 $Comp
-L Mechanical:MountingHole H1
+L microtaur-teensy41-rescue:MountingHole-Mechanical H1
 U 1 1 608B9565
 P 750 6800
@@
 $EndComp
 $Comp
-L Connector_Generic:Conn_01x02 MPOW1
+L microtaur-teensy41-rescue:Conn_01x02-Connector_Generic MPOW1
 U 1 1 608C3689
 P 9050 1200
@@
 $EndComp
 $Comp
-L Connector_Generic:Conn_01x02 MPOW2
+L microtaur-teensy41-rescue:Conn_01x02-Connector_Generic MPOW2
 U 1 1 608CC08E
 P 9050 1500
@@
 $EndComp
 $Comp
-L Connector_Generic:Conn_01x02 MPOW3
+L microtaur-teensy41-rescue:Conn_01x02-Connector_Generic MPOW3
 U 1 1 608CC4B3
 P 9050 1800
@@
 $EndComp
 $Comp
-L Connector_Generic:Conn_01x02 MPOW4
+L microtaur-teensy41-rescue:Conn_01x02-Connector_Generic MPOW4
 U 1 1 608CC6EE
 P 9050 2100
@@
 $EndComp
 $Comp
-L Connector_Generic:Conn_01x02 MPOW5
+L microtaur-teensy41-rescue:Conn_01x02-Connector_Generic MPOW5
 U 1 1 608CE9C3
 P 9050 2400
@@
 $EndComp
 $Comp
-L Connector_Generic:Conn_01x02 MPOW6
+L microtaur-teensy41-rescue:Conn_01x02-Connector_Generic MPOW6
 U 1 1 608CE9C9
 P 9050 2700
@@
 $EndComp
 $Comp
-L Connector_Generic:Conn_01x02 MPOW7
+L microtaur-teensy41-rescue:Conn_01x02-Connector_Generic MPOW7
 U 1 1 608CE9CF
 P 9050 3000
@@
 $EndComp
 $Comp
-L Connector_Generic:Conn_01x02 MPOW8
+L microtaur-teensy41-rescue:Conn_01x02-Connector_Generic MPOW8
 U 1 1 608CE9D5
 P 9050 3300
@@
 $EndComp
 $Comp
-L power:Vdrive #PWR0114
+L microtaur-teensy41-rescue:Vdrive-power #PWR0114
 U 1 1 608E45DF
 P 10800 5650
@@
 D-
 $Comp
-L power:GND #PWR02
+L microtaur-teensy41-rescue:GND-power #PWR02
 U 1 1 6091D07A
 P 3100 4550
@@
 $EndComp
 $Comp
-L power:GND #PWR01
+L microtaur-teensy41-rescue:GND-power #PWR01
 U 1 1 6091D5BC
 P 3000 4550
@@
 	4150 4050 4350 4050
 $Comp
-L power:GND #PWR03
+L microtaur-teensy41-rescue:GND-power #PWR03
 U 1 1 60925E27
 P 4350 4250
@@
 $EndComp
 $Comp
-L power:GND #PWR04
+L microtaur-teensy41-rescue:GND-power #PWR04
 U 1 1 6092511C
 P 4350 4350
@@
 $EndComp
 $Comp
-L power:Vdrive #PWR0115
+L microtaur-teensy41-rescue:Vdrive-power #PWR0115
 U 1 1 608EB897
 P 8850 1300
@@
 $EndComp
 $Comp
-L power:GND #PWR0113
+L microtaur-teensy41-rescue:GND-power #PWR0113
 U 1 1 608DE0A0
 P 8850 1200
@@
 $EndComp
 $Comp
-L power:Vdrive #PWR0116
+L microtaur-teensy41-rescue:Vdrive-power #PWR0116
 U 1 1 6093B156
 P 8850 1600
@@
 $EndComp
 $Comp
-L power:GND #PWR0117
+L microtaur-teensy41-rescue:GND-power #PWR0117
 U 1 1 6093B15C
 P 8850 1500
@@
 $EndComp
 $Comp
-L power:Vdrive #PWR0118
+L microtaur-teensy41-rescue:Vdrive-power #PWR0118
 U 1 1 6093DD87
 P 8850 1900
@@
 $EndComp
 $Comp
-L power:GND #PWR0119
+L microtaur-teensy41-rescue:GND-power #PWR0119
 U 1 1 6093DD8D
 P 8850 1800
@@
 $EndComp
 $Comp
-L power:Vdrive #PWR0120
+L microtaur-teensy41-rescue:Vdrive-power #PWR0120
 U 1 1 6093DD93
 P 8850 2200
@@
 $EndComp
 $Comp
-L power:GND #PWR0121
+L microtaur-teensy41-rescue:GND-power #PWR0121
 U 1 1 6093DD99
 P 8850 2100
@@
 $EndComp
 $Comp
-L power:Vdrive #PWR0122
+L microtaur-teensy41-rescue:Vdrive-power #PWR0122
 U 1 1 60941308
 P 8850 2500
@@
 $EndComp
 $Comp
-L power:GND #PWR0123
+L microtaur-teensy41-rescue:GND-power #PWR0123
 U 1 1 6094130E
 P 8850 2400
@@
 $EndComp
 $Comp
-L power:Vdrive #PWR0124
+L microtaur-teensy41-rescue:Vdrive-power #PWR0124
 U 1 1 60941314
 P 8850 2800
@@
 $EndComp
 $Comp
-L power:GND #PWR0125
+L microtaur-teensy41-rescue:GND-power #PWR0125
 U 1 1 6094131A
 P 8850 2700
@@
 $EndComp
 $Comp
-L power:Vdrive #PWR0126
+L microtaur-teensy41-rescue:Vdrive-power #PWR0126
 U 1 1 60944C09
 P 8850 3100
@@
 $EndComp
 $Comp
-L power:GND #PWR0127
+L microtaur-teensy41-rescue:GND-power #PWR0127
 U 1 1 60944C0F
 P 8850 3000
@@
 $EndComp
 $Comp
-L power:Vdrive #PWR0128
+L microtaur-teensy41-rescue:Vdrive-power #PWR0128
 U 1 1 60944C15
 P 8850 3400
@@
 $EndComp
 $Comp
-L power:GND #PWR0129
+L microtaur-teensy41-rescue:GND-power #PWR0129
 U 1 1 60944C1B
 P 8850 3300
@@
 $EndComp
 $Comp
-L Connector_Generic:Conn_01x04 IMU1
+L microtaur-teensy41-rescue:Conn_01x04-Connector_Generic IMU1
 U 1 1 6095C393
 P 5550 6050
@@
 Connection ~ 9400 5450
 $Comp
-L Regulator_Linear:LM7805_TO220 U3
+L microtaur-teensy41-rescue:LM7805_TO220-Regulator_Linear U3
 U 1 1 6097103B
 P 9100 5450
